Commit message: add caster model

File: urdf/3dmodel.urdf (robot description, URDF)
Before this commit: robot micro_motor, 1 links, 0 joints
Links:
- link base_link: geometry visual mesh filename=package://urdf/meshes/pololu-ball-caster-with-0-375in-ball.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

File: urdf/roundrobot.urdf (robot description, URDF)
Before this commit: robot round_robot, 1 links, 1 joints
Links:
- added link caster, mass 0.004; collision box size=0.0191 0.0121 0.0101; visual mesh filename=package://urdf/meshes/pololu-ball-caster-with-0-375in-ball.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
- link chassis: geometry collision cylinder length=0.003 radius=0.0635; visual cylinder length=0.003 radius=0.0635
Joints:
- joint chassis2caster: origin xyz=0.125 0 -0.05 rpy=0 0 0 -> xyz=0.054 0 -0.003 rpy=0 3.141592653589793 1.5707963267948966

Commit message: add motors and wheels

File: urdf/3dmodel.urdf (robot description, URDF)
Before this commit: robot micro_motor, 1 links, 0 joints
Links:
- link base_link: geometry visual mesh filename=package://urdf/meshes/micro-metal-gearmotor-with-1086-brack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

File: urdf/roundrobot.urdf (robot description, URDF)
Before this commit: robot round_robot, 2 links, 1 joints
Links:
- added link left_motor, mass 0.0095; collision box size=0.038 0.012 0.010; visual mesh filename=package://urdf/meshes/micro-metal-gearmotor-with-1086-brack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
- added link left_wheel, mass 0.019; collision cylinder length=0.019 radius=0.021; visual mesh filename=package://urdf/meshes/pololu-wheel-42x19mm.dae
- added link right_motor, mass 0.0095; collision box size=0.038 0.012 0.010; visual mesh filename=package://urdf/meshes/micro-metal-gearmotor-with-1086-brack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
- added link right_wheel, mass 0.019; collision cylinder length=0.019 radius=0.021; visual mesh filename=package://urdf/meshes/pololu-wheel-42x19mm.dae
Joints:
- added joint chassis2left_motor: type fixed, parent chassis, child left_motor, origin xyz=0 0.033 0.00875 rpy=1.5707963267948966 0 1.5707963267948966
- added joint chassis2right_motor: type fixed, parent chassis, child right_motor, origin xyz=0 -0.033 0.00875 rpy=1.5707963267948966 0 -1.5707963267948966
- added joint left_motor2left_wheel: type continuous, parent left_motor, child left_wheel, origin xyz=0.016 0 0 rpy=0 1.5707963267948966 0, axis 1 0 0
- added joint right_motor2right_wheel: type continuous, parent right_motor, child right_wheel, origin xyz=0.016 0 0 rpy=0 -1.5707963267948966 0, axis 1 0 0
